Commit message: 更新STL文件，解决大部分显示问题，base_link显示仍有问题

File: src/mygo_robot_description/urdf/arm.xacro (robot description, xacro)
@@ -1,17 +1,17 @@
 <?xml version="1.0"?>
 <robot xmlns:xacro="http://www.ros.org/wiki/xacro">
-  <xacro:macro name="mygo_arm" params="prefix:=''>
+  <xacro:macro name="mygo_arm" params="prefix:=''">
     <link name="${prefix}base_link">
       <visual>
-        <origin xyz="0 0 0.022" rpy="0 0 0"/>
+        <origin xyz="0 0 0" rpy="0 0 0"/>
         <geometry>
-          <box size="0.08 0.08 0.044"/>
+          <mesh filename="package://mygo_robot_description/meshes/base_link.STL"/>
         </geometry>
         <material name="gray"/>
       </visual>
       <collision>
-        <origin xyz="0 0 0.022" rpy="0 0 0"/>
+        <origin xyz="0 0 0" rpy="0 0 0"/>
         <geometry>
-          <box size="0.08 0.08 0.044"/>
+          <mesh filename="package://mygo_robot_description/meshes/base_link.STL"/>
         </geometry>
       </collision>
@@ -19,14 +19,14 @@
     <link name="${prefix}link1">
       <visual>
-        <origin xyz="0 0 0.03" rpy="0 0 0"/>
+        <origin xyz="0 0 0" rpy="0 0 0"/>
         <geometry>
-          <cylinder length="0.06" radius="0.024"/>
+          <mesh filename="package://mygo_robot_description/meshes/link1.STL"/>
         </geometry>
         <material name="white"/>
       </visual>
       <collision>
-        <origin xyz="0 0 0.03" rpy="0 0 0"/>
+        <origin xyz="0 0 0" rpy="0 0 0"/>
         <geometry>
-          <cylinder length="0.06" radius="0.024"/>
+          <mesh filename="package://mygo_robot_description/meshes/link1.STL"/>
         </geometry>
       </collision>
@@ -40,14 +40,14 @@
     <link name="${prefix}link2">
       <visual>
-        <origin xyz="0 -0.052 0" rpy="1.5708 0 0"/>
+        <origin xyz="0 0 0" rpy="0 0 0"/>
         <geometry>
-          <cylinder length="0.105" radius="0.018"/>
+          <mesh filename="package://mygo_robot_description/meshes/link2.STL"/>
         </geometry>
         <material name="dark_gray"/>
       </visual>
       <collision>
-        <origin xyz="0 -0.052 0" rpy="1.5708 0 0"/>
+        <origin xyz="0 0 0" rpy="0 0 0"/>
         <geometry>
-          <cylinder length="0.105" radius="0.018"/>
+          <mesh filename="package://mygo_robot_description/meshes/link2.STL"/>
         </geometry>
       </collision>
@@ -62,14 +62,14 @@
     <link name="${prefix}link3">
       <visual>
-        <origin xyz="0 -0.05 0" rpy="1.5708 0 0"/>
+        <origin xyz="0 0 0" rpy="0 0 0"/>
         <geometry>
-          <cylinder length="0.10" radius="0.017"/>
+          <mesh filename="package://mygo_robot_description/meshes/link3.STL"/>
         </geometry>
         <material name="dark_gray"/>
       </visual>
       <collision>
-        <origin xyz="0 -0.05 0" rpy="1.5708 0 0"/>
+        <origin xyz="0 0 0" rpy="0 0 0"/>
         <geometry>
-          <cylinder length="0.10" radius="0.017"/>
+          <mesh filename="package://mygo_robot_description/meshes/link3.STL"/>
         </geometry>
       </collision>
@@ -84,14 +84,14 @@
     <link name="${prefix}link4">
       <visual>
-        <origin xyz="0 -0.047 0" rpy="1.5708 0 0"/>
+        <origin xyz="0 0 0" rpy="0 0 0"/>
         <geometry>
-          <cylinder length="0.094" radius="0.016"/>
+          <mesh filename="package://mygo_robot_description/meshes/link4.STL"/>
         </geometry>
         <material name="gray"/>
       </visual>
       <collision>
-        <origin xyz="0 -0.047 0" rpy="1.5708 0 0"/>
+        <origin xyz="0 0 0" rpy="0 0 0"/>
         <geometry>
-          <cylinder length="0.094" radius="0.016"/>
+          <mesh filename="package://mygo_robot_description/meshes/link4.STL"/>
         </geometry>
       </collision>
@@ -106,14 +106,14 @@
     <link name="${prefix}link5">
       <visual>
-        <origin xyz="-0.02 -0.04 -0.02" rpy="1.5708 0 0"/>
+        <origin xyz="0 0 0" rpy="0 0 0"/>
         <geometry>
-          <cylinder length="0.08" radius="0.015"/>
+          <mesh filename="package://mygo_robot_description/meshes/link5.STL"/>
         </geometry>
         <material name="white"/>
       </visual>
       <collision>
-        <origin xyz="-0.02 -0.04 -0.02" rpy="1.5708 0 0"/>
+        <origin xyz="0 0 0" rpy="0 0 0"/>
         <geometry>
-          <cylinder length="0.08" radius="0.015"/>
+          <mesh filename="package://mygo_robot_description/meshes/link5.STL"/>
         </geometry>
       </collision>

File: src/mygo_robot_description/urdf/gripper.xacro (robot description, xacro)
@@ -4,14 +4,14 @@
     <link name="${prefix}end_link1">
       <visual>
-        <origin xyz="0 -0.03 -0.02" rpy="1.5708 0 0"/>
+        <origin xyz="0 0 0" rpy="0 0 0"/>
         <geometry>
-          <box size="0.012 0.06 0.01"/>
+          <mesh filename="package://mygo_robot_description/meshes/end link1.STL"/>
         </geometry>
         <material name="white"/>
       </visual>
       <collision>
-        <origin xyz="0 -0.03 -0.02" rpy="1.5708 0 0"/>
+        <origin xyz="0 0 0" rpy="0 0 0"/>
         <geometry>
-          <box size="0.012 0.06 0.01"/>
+          <mesh filename="package://mygo_robot_description/meshes/end link1.STL"/>
         </geometry>
       </collision>
@@ -26,14 +26,14 @@
     <link name="${prefix}end_link2">
       <visual>
-        <origin xyz="0 0.03 -0.02" rpy="1.5708 0 0"/>
+        <origin xyz="0 0 0" rpy="0 0 0"/>
         <geometry>
-          <box size="0.012 0.06 0.01"/>
+          <mesh filename="package://mygo_robot_description/meshes/end link2.STL"/>
         </geometry>
         <material name="white"/>
       </visual>
       <collision>
-        <origin xyz="0 0.03 -0.02" rpy="1.5708 0 0"/>
+        <origin xyz="0 0 0" rpy="0 0 0"/>
         <geometry>
-          <box size="0.012 0.06 0.01"/>
+          <mesh filename="package://mygo_robot_description/meshes/end link2.STL"/>
         </geometry>
       </collision>

Commit message: 修正关节限位，等待base_linkSTL模型

File: src/mygo_robot_description/urdf/arm.xacro (robot description, xacro)
@@ -58,5 +58,5 @@
       <child link="${prefix}link2"/>
       <axis xyz="0 0 -1"/>
-      <limit lower="-3.14159" upper="3.14159" effort="10" velocity="1"/>
+      <limit lower="-2.35619" upper="2.35619" effort="10" velocity="1"/>
     </joint>
     <link name="${prefix}link3">
@@ -80,5 +80,5 @@
       <child link="${prefix}link3"/>
       <axis xyz="0 0.066173 -0.99781"/>
-      <limit lower="-3.14159" upper="3.14159" effort="10" velocity="1"/>
+      <limit lower="-2.35619" upper="2.35619" effort="10" velocity="1"/>
     </joint>
     <link name="${prefix}link4">
@@ -102,5 +102,5 @@
       <child link="${prefix}link4"/>
       <axis xyz="0 0.066173 -0.99781"/>
-      <limit lower="-3.14159" upper="3.14159" effort="10" velocity="1"/>
+      <limit lower="-2.35619" upper="2.35619" effort="10" velocity="1"/>
     </joint>
     <link name="${prefix}link5">
@@ -124,5 +124,5 @@
       <child link="${prefix}link5"/>
       <axis xyz="0 0 -1"/>
-      <limit lower="-3.14159" upper="3.14159" effort="10" velocity="1"/>
+      <limit lower="-2.35619" upper="2.35619" effort="10" velocity="1"/>
     </joint>
   </xacro:macro>

Commit message: 修复机械臂个别舵机角度定义相反的问题

File: src/mygo_robot_description/urdf/arm.xacro (robot description, xacro)
@@ -57,5 +57,5 @@
       <parent link="${prefix}link1"/>
       <child link="${prefix}link2"/>
-      <axis xyz="0 0 -1"/>
+      <axis xyz="0 0 1"/>
       <limit lower="-2.35619" upper="2.35619" effort="10" velocity="1"/>
     </joint>
@@ -79,5 +79,5 @@
       <parent link="${prefix}link2"/>
       <child link="${prefix}link3"/>
-      <axis xyz="0 0.066173 -0.99781"/>
+      <axis xyz="0 -0.066173 0.99781"/>
       <limit lower="-2.35619" upper="2.35619" effort="10" velocity="1"/>
     </joint>
@@ -123,5 +123,5 @@
       <parent link="${prefix}link4"/>
       <child link="${prefix}link5"/>
-      <axis xyz="0 0 -1"/>
+      <axis xyz="0 0 1"/>
       <limit lower="-2.35619" upper="2.35619" effort="10" velocity="1"/>
     </joint>

File: src/mygo_robot_description/urdf/gripper.xacro (robot description, xacro)
@@ -21,5 +21,5 @@
       <parent link="${prefix}${parent}"/>
       <child link="${prefix}end_link1"/>
-      <axis xyz="0 -0.99836 0.057228"/>
+      <axis xyz="0 0.99836 -0.057228"/>
       <limit lower="-3.14159" upper="3.14159" effort="10" velocity="1"/>
     </joint>
@@ -43,5 +43,5 @@
       <parent link="${prefix}${parent}"/>
       <child link="${prefix}end_link2"/>
-      <axis xyz="0 0 -1"/>
+      <axis xyz="0 0 1"/>
       <limit lower="-3.14159" upper="3.14159" effort="10" velocity="1"/>
       <mimic joint="${prefix}end_joint1" multiplier="-1" offset="0"/>

Commit message: 修正baselink的STL文件

File: src/mygo_robot_description/urdf/arm.xacro (robot description, xacro)
@@ -4,5 +4,5 @@
     <link name="${prefix}base_link">
       <visual>
-        <origin xyz="0 0 0" rpy="0 0 0"/>
+        <origin xyz="0.02 0 0" rpy="0.02 0 0"/>
         <geometry>
           <mesh filename="package://mygo_robot_description/meshes/base_link.STL"/>
@@ -11,5 +11,5 @@
       </visual>
       <collision>
-        <origin xyz="0 0 0" rpy="0 0 0"/>
+        <origin xyz="0.02 0 0" rpy="0.02 0 0"/>
         <geometry>
           <mesh filename="package://mygo_robot_description/meshes/base_link.STL"/>
